File: romboard.brd (EAGLE design)
At the start: 86 x 59 mm, 13 parts

Commit message: Add licence to schematic, board
Other:
- board text added: "CC BY-SA 3.0"
Changed lines of the file:
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@@
 <wire x1="82.55" y1="54.61" x2="81.28" y2="53.34" width="0.4064" layer="51"/>
 <rectangle x1="11.43" y1="45.72" x2="12.7" y2="47.625" layer="52"/>
+<text x="76.2" y="7.62" size="1.778" layer="51" rot="MR90">CC BY-SA 3.0</text>
 </plain>
 <attributes>
